Commit message: Split the bot urdf description into several files

File: bot_description/urdf/bot.urdf.xacro (robot description, xacro)
@@ -55,44 +55,6 @@
     <xacro:box_inertia m="${base_mass}" x="${base_length}" y="${base_width}" z="${base_height}"/>
   </link>
-  <xacro:macro name="wheel" params="prefix reflect">
-    <link name="${prefix}_wheel">
-      <visual>
-        <origin xyz="0 0 0" rpy="${pi/2} 0 0" />
-        <geometry>
-          <cylinder radius="${wheel_radius}" length="${wheel_width}"/>
-        </geometry>
-        <material name="black"/>
-      </visual>
-      <collision>
-        <origin xyz="0 0 0" rpy="${pi/2} 0 0" />
-        <geometry>
-          <cylinder radius="${wheel_radius}" length="${wheel_width}"/>
-        </geometry>
-      </collision>
-      <xacro:cylinder_inertia m="${wheel_mass}" r="${wheel_radius}" h="${wheel_width}"/>
-    </link>
-    <joint name="${prefix}_wheel_joint" type="continuous">
-      <axis xyz="0 1 0" rpy="0 0 0" />
-      <parent link="base_link"/>
-      <child link="${prefix}_wheel"/>
-      <origin xyz="${base_length/3.6} ${base_width/2*reflect + wheel_width/2*reflect} -${base_height/2}" rpy="0 0 0"/>
-    </joint>
-    <gazebo reference="${prefix}_wheel">
-      <mu1 value="200.0"/>
-      <mu2 value="100.0"/>
-      <kp value="10000000.0" />
-      <kd value="1.0" />
-      <material>Gazebo/Black</material>
-    </gazebo>
-    <transmission name="${prefix}_wheel_trans">
-      <type>transmission_interface/SimpleTransmission</type>
-      <actuator name="${prefix}_wheel_motor">
-        <mechanicalReduction>1</mechanicalReduction>
-      </actuator>
-      <joint name="${prefix}_wheel_joint">
-        <hardwareInterface>hardware_interface/VelocityJointInterface</hardwareInterface>
-      </joint>
-    </transmission>
-  </xacro:macro>
+  <xacro:include filename="$(find bot_description)/urdf/camera.urdf.xacro" />
+  <xacro:include filename="$(find bot_description)/urdf/wheel.urdf.xacro" />
   <xacro:wheel prefix="right" reflect="1"/>
   <xacro:wheel prefix="left" reflect="-1"/>

Commit message: Make SLAM work in simulation

File: bot_description/urdf/bot.urdf.xacro (robot description, xacro)
@@ -1,9 +1,9 @@
 <?xml version="1.0"?>
 <robot name="rosbot" xmlns:xacro="http://ros.org/wiki/xacro">
-  <xacro:property name="base_mass" value="0.9" />
+  <xacro:property name="base_mass" value="10.0" />
   <xacro:property name="base_length" value="0.145" />
   <xacro:property name="base_width"  value="0.1" />
   <xacro:property name="base_height" value="0.11" />
-  <xacro:property name="wheel_mass" value="0.01" />
+  <xacro:property name="wheel_mass" value="3.0" />
   <xacro:property name="wheel_radius" value="0.025" />
   <xacro:property name="wheel_width" value="0.005" />
@@ -52,4 +52,14 @@
         <box size="${base_length} ${base_width} ${base_height}"/>
       </geometry>
+      <surface>
+        <friction>
+          <ode>
+            <mu>0</mu>
+            <mu2>0</mu2>
+            <slip1>1.0</slip1>
+            <slip2>1.0</slip2>
+          </ode>
+        </friction>
+      </surface>
     </collision>
     <xacro:box_inertia m="${base_mass}" x="${base_length}" y="${base_width}" z="${base_height}"/>

File: bot_description/urdf/camera.urdf.xacro (robot description, xacro)
@@ -18,5 +18,5 @@
 </link>
 <joint name="top_camera_joint" type="fixed">
-  <origin xyz="0.0  0.0 ${base_height/2 + 0.02}" rpy="0 0 0" />
+  <origin xyz="${base_length/2 - 0.02} 0.0 ${base_height/2 + 0.02}" rpy="0 0 0" />
   <parent link="base_link" />
   <child link="top_camera"/>
@@ -26,8 +26,8 @@
    <update_rate>30.0</update_rate>
    <camera name="head">
-     <horizontal_fov>1.3962634</horizontal_fov>
+     <horizontal_fov>1.57</horizontal_fov>
      <image>
-       <width>800</width>
-       <height>600</height>
+       <width>640</width>
+       <height>480</height>
        <format>R8G8B8</format>
      </image>
@@ -44,10 +44,10 @@
    <plugin name="camera_controller" filename="libgazebo_ros_camera.so">
      <alwaysOn>true</alwaysOn>
-     <updateRate>30.0</updateRate>
+     <updateRate>0.0</updateRate>
      <cameraName>rosbot/main_camera</cameraName>
      <imageTopicName>image_raw</imageTopicName>
      <cameraInfoTopicName>camera_info</cameraInfoTopicName>
      <frameName>camera_link_optical</frameName>
-     <hackBaseline>0.0</hackBaseline>
+     <hackBaseline>0.07</hackBaseline>
      <distortionK1>0.0</distortionK1>
      <distortionK2>0.0</distortionK2>
@@ -55,8 +55,10 @@
      <distortionT1>0.0</distortionT1>
      <distortionT2>0.0</distortionT2>
-     <CxPrime>0</CxPrime>
-     <Cx>0.0</Cx>
-     <Cy>0.0</Cy>
-     <focalLength>0.0</focalLength>
+<!--
+     <CxPrime>320</CxPrime>
+     <Cx>320</Cx>
+     <Cy>240</Cy>
+     <focalLength>381</focalLength>
+-->
    </plugin>
  </sensor>

File: bot_description/urdf/wheel.urdf.xacro (robot description, xacro)
@@ -23,4 +23,6 @@
     <child link="${prefix}_wheel"/>
     <origin xyz="${base_length/3.6} ${base_width/2*reflect + wheel_width/2*reflect} -${base_height/2}" rpy="0 0 0"/>
+    <limit effort="10000" velocity="1000"/>
+    <joint_properties damping="0.0" friction="0.0"/>
   </joint>
   <gazebo reference="${prefix}_wheel">

Commit message: Add 2d navigation stack

File: bot_description/urdf/bot.urdf.xacro (robot description, xacro)
@@ -67,6 +67,6 @@
   <xacro:include filename="$(find bot_description)/urdf/camera.urdf.xacro" />
   <xacro:include filename="$(find bot_description)/urdf/wheel.urdf.xacro" />
-  <xacro:wheel prefix="right" reflect="1"/>
-  <xacro:wheel prefix="left" reflect="-1"/>
+  <xacro:wheel prefix="left" reflect="1"/>
+  <xacro:wheel prefix="right" reflect="-1"/>
   <link name="rear_wheel">
     <visual>

File: bot_description/urdf/wheel.urdf.xacro (robot description, xacro)
@@ -23,5 +23,5 @@
     <child link="${prefix}_wheel"/>
     <origin xyz="${base_length/3.6} ${base_width/2*reflect + wheel_width/2*reflect} -${base_height/2}" rpy="0 0 0"/>
-    <limit effort="10000" velocity="1000"/>
+    <limit effort="10000" velocity="10"/>
     <joint_properties damping="0.0" friction="0.0"/>
   </joint>
